Commit message: Gazebo_launch_success

File: src/nav4wbot_description/urdf/nav4wbot.urdf.xacro (robot description, xacro)
@@ -1,6 +1,10 @@
 <?xml version="1.0"?>
 <robot xmlns:xacro="http://ros.org/wiki/xacro" name="nav4wbot">
+  <!-- ============ Properties ============ -->
   <xacro:property name="wheel_radius" value="0.1"/>
-  <xacro:property name="wheel_base" value="0.4"/>
+  <xacro:property name="wheel_thickness" value="0.05"/>
+  <xacro:property name="wheel_base" value="0.4"/>   <!-- front-back distance -->
+  <xacro:property name="track_width" value="0.35"/>  <!-- left-right distance -->
+  <!-- ============ Base Link ============ -->
   <link name="base_link">
     <visual>
@@ -8,35 +12,103 @@
         <box size="0.5 0.3 0.1"/>
       </geometry>
+      <origin xyz="0 0 0.1" rpy="0 0 0"/>
       <material name="grey">
         <color rgba="0.5 0.5 0.5 1.0"/>
       </material>
     </visual>
+    <collision>
+      <geometry>
+        <box size="0.5 0.3 0.1"/>
+      </geometry>
+      <origin xyz="0 0 0.1" rpy="0 0 0"/>
+    </collision>
+    <inertial>
+      <mass value="10.0"/>
+    </inertial>
   </link>
-  <!-- Four wheels -->
+  <!-- ============ Wheel Macro ============ -->
   <xacro:macro name="wheel" params="name x y">
     <link name="${name}">
       <visual>
         <geometry>
-          <cylinder radius="${wheel_radius}" length="0.05"/>
+          <cylinder radius="${wheel_radius}" length="${wheel_thickness}"/>
         </geometry>
-        <material name="black"/>
+        <!-- Rotate cylinder so axis aligns with wheel axle -->
+        <origin xyz="0 0 0" rpy="1.5708 0 0"/> <!-- rotate 90deg about x -->
+        <material name="black">
+          <color rgba="0 0 0 1"/>
+        </material>
       </visual>
+      <collision>
+        <geometry>
+          <cylinder radius="${wheel_radius}" length="${wheel_thickness}"/>
+        </geometry>
+        <origin xyz="0 0 0" rpy="1.5708 0 0"/>
+      </collision>
+      <inertial>
+        <mass value="1.0"/>
+        <inertia ixx="0.01" ixy="0.0" ixz="0.0"
+                 iyy="0.01" iyz="0.0"
+                 izz="0.01"/>
+      </inertial>
     </link>
     <joint name="${name}_joint" type="continuous">
       <parent link="base_link"/>
       <child link="${name}"/>
-      <origin xyz="${x} ${y} 0" rpy="0 0 0"/>
-      <axis xyz="0 1 0"/>
+      <origin xyz="${x} ${y} ${wheel_radius}" rpy="0 0 0"/>
+      <axis xyz="0 1 0"/> <!-- wheel rotates around y-axis -->
     </joint>
   </xacro:macro>
-  <xacro:wheel name="left_front_wheel" x="0.2" y="0.15"/>
-  <xacro:wheel name="left_rear_wheel" x="-0.2" y="0.15"/>
-  <xacro:wheel name="right_front_wheel" x="0.2" y="-0.15"/>
-  <xacro:wheel name="right_rear_wheel" x="-0.2" y="-0.15"/>
-  <!-- Diff drive controller plugin -->
+  <!-- ============ Wheels ============ -->
+  <xacro:wheel name="left_front_wheel"  x="0.2"  y="0.175"/>
+  <xacro:wheel name="left_rear_wheel"   x="-0.2" y="0.175"/>
+  <xacro:wheel name="right_front_wheel" x="0.2"  y="-0.175"/>
+  <xacro:wheel name="right_rear_wheel"  x="-0.2" y="-0.175"/>
+  <!-- ============ Lidar Sensor ============ -->
+  <link name="lidar_link">
+    <visual>
+      <geometry>
+        <cylinder radius="0.05" length="0.1"/>
+      </geometry>
+      <origin xyz="0 0 0.05" rpy="0 0 0"/>
+      <material name="blue">
+        <color rgba="0.2 0.2 0.8 1"/>
+      </material>
+    </visual>
+  </link>
+  <joint name="lidar_joint" type="fixed">
+    <parent link="base_link"/>
+    <child link="lidar_link"/>
+    <origin xyz="0 0 0.15" rpy="0 0 0"/>
+  </joint>
+  <!-- Gazebo plugin for Lidar -->
+  <gazebo reference="lidar_link">
+    <sensor type="gpu_ray" name="lidar_sensor">
+      <update_rate>10</update_rate>
+      <ray>
+        <scan>
+          <horizontal>
+            <samples>720</samples>
+            <resolution>1</resolution>
+            <min_angle>-1.5708</min_angle>
+            <max_angle>1.5708</max_angle>
+          </horizontal>
+        </scan>
+        <range>
+          <min>0.12</min>
+          <max>10.0</max>
+          <resolution>0.01</resolution>
+        </range>
+      </ray>
+      <plugin name="gazebo_ros_laser" filename="libgazebo_ros_ray_sensor.so"/>
+    </sensor>
+  </gazebo>
+  <!-- ============ Diff Drive Plugin ============ -->
   <gazebo>
     <plugin name="diff_drive_controller" filename="libgazebo_ros2_control_differential_drive.so">
       <left_joint>left_front_wheel_joint</left_joint>
+      <left_joint>left_rear_wheel_joint</left_joint>
       <right_joint>right_front_wheel_joint</right_joint>
+      <right_joint>right_rear_wheel_joint</right_joint>
       <wheel_separation>${wheel_base}</wheel_separation>
       <wheel_radius>${wheel_radius}</wheel_radius>

Commit message: urdf_cleanup

File: src/nav4wbot_description/urdf/nav4wbot.urdf.xacro (robot description, xacro)
@@ -1,11 +1,52 @@
 <?xml version="1.0"?>
 <robot xmlns:xacro="http://ros.org/wiki/xacro" name="nav4wbot">
-  <!-- ============ Properties ============ -->
-  <xacro:property name="wheel_radius" value="0.1"/>
-  <xacro:property name="wheel_thickness" value="0.05"/>
-  <xacro:property name="wheel_base" value="0.4"/>   <!-- front-back distance -->
-  <xacro:property name="track_width" value="0.35"/>  <!-- left-right distance -->
-  <!-- ============ Base Link ============ -->
+  <!-- Properties for dimensions -->
+  <xacro:property name="PI" value="3.14159" />
+  <xacro:property name="wheel_radius" value="0.1" />
+  <xacro:property name="wheel_thickness" value="0.05" />
+  <xacro:property name="wheel_base" value="0.4" />          <!-- front-back distance(change) -->
+  <xacro:property name="track_width" value="0.35" />        <!-- left-right distance(change) -->
+  <!-- Macros Definations -->
+  <!-- Intertial Macro -->
+  <xacro:macro name="default_interial" params="mass">
+    <inertial>
+      <mass value="${mass}"/>
+      <inertia ixx="0.01" ixy="0.0" ixz="0.0"
+               iyy="0.01" iyz="0.0"
+               izz="0.01"/>
+    </inertial>
+  </xacro:macro>
+  <!--  Wheel Macro  -->
+  <xacro:macro name="wheel" params="name x y">
+    <link name="${name}">
+      <xacro:default_interial mass="1.0"/>
+      <visual>
+        <geometry>
+          <cylinder radius="${wheel_radius}" length="${wheel_thickness}"/>
+        </geometry>
+        <origin xyz="0 0 0" rpy="${PI/2} 0 0"/>
+        <material name="black">
+          <color rgba="0 0 0 1"/>
+        </material>
+      </visual>
+      <collision>
+        <geometry>
+          <cylinder radius="${wheel_radius}" length="${wheel_thickness}"/>
+        </geometry>
+        <origin xyz="0 0 0" rpy="${PI/2} 0 0"/>
+      </collision>
+    </link>
+    <joint name="${name}_joint" type="continuous">
+      <parent link="base_link"/>
+      <child link="${name}"/>
+      <origin xyz="${x} ${y} ${wheel_radius}" rpy="0 0 0"/>
+      <axis xyz="0 1 0"/>
+    </joint>
+  </xacro:macro>
+  <!-- Robot Description -->
+  <link name="world"/>
+  <!-- Base Link -->
   <link name="base_link">
+    <xacro:default_interial mass="10.0"/>
     <visual>
       <geometry>
@@ -23,42 +64,11 @@
       <origin xyz="0 0 0.1" rpy="0 0 0"/>
     </collision>
-    <inertial>
-      <mass value="10.0"/>
-    </inertial>
   </link>
-  <!-- ============ Wheel Macro ============ -->
-  <xacro:macro name="wheel" params="name x y">
-    <link name="${name}">
-      <visual>
-        <geometry>
-          <cylinder radius="${wheel_radius}" length="${wheel_thickness}"/>
-        </geometry>
-        <!-- Rotate cylinder so axis aligns with wheel axle -->
-        <origin xyz="0 0 0" rpy="1.5708 0 0"/> <!-- rotate 90deg about x -->
-        <material name="black">
-          <color rgba="0 0 0 1"/>
-        </material>
-      </visual>
-      <collision>
-        <geometry>
-          <cylinder radius="${wheel_radius}" length="${wheel_thickness}"/>
-        </geometry>
-        <origin xyz="0 0 0" rpy="1.5708 0 0"/>
-      </collision>
-      <inertial>
-        <mass value="1.0"/>
-        <inertia ixx="0.01" ixy="0.0" ixz="0.0"
-                 iyy="0.01" iyz="0.0"
-                 izz="0.01"/>
-      </inertial>
-    </link>
-    <joint name="${name}_joint" type="continuous">
-      <parent link="base_link"/>
-      <child link="${name}"/>
-      <origin xyz="${x} ${y} ${wheel_radius}" rpy="0 0 0"/>
-      <axis xyz="0 1 0"/> <!-- wheel rotates around y-axis -->
-    </joint>
-  </xacro:macro>
-  <!-- ============ Wheels ============ -->
+  <joint name="virtual_joint" type="fixed">
+    <parent link="world"/>
+    <child link="base_link"/>
+    <origin xyz="0 0 0" rpy="0 0 0"/>
+  </joint>
+  <!--  Wheels  -->
   <xacro:wheel name="left_front_wheel"  x="0.2"  y="0.175"/>
   <xacro:wheel name="left_rear_wheel"   x="-0.2" y="0.175"/>
@@ -67,4 +77,5 @@
   <!-- ============ Lidar Sensor ============ -->
   <link name="lidar_link">
+    <xacro:default_interial mass="0.5"/>
     <visual>
       <geometry>
@@ -84,4 +95,6 @@
   <!-- Gazebo plugin for Lidar -->
   <gazebo reference="lidar_link">
+    <!-- Note my gazebo is ign gazebo, so change the plugin as needed -->
+    <plugin name="gazebo_ros_laser" filename="libgazebo_ros_ray_sensor.so"/>
     <sensor type="gpu_ray" name="lidar_sensor">
       <update_rate>10</update_rate>
@@ -101,5 +114,4 @@
         </range>
       </ray>
-      <plugin name="gazebo_ros_laser" filename="libgazebo_ros_ray_sensor.so"/>
     </sensor>
   </gazebo>
@@ -111,5 +123,6 @@
       <right_joint>right_front_wheel_joint</right_joint>
       <right_joint>right_rear_wheel_joint</right_joint>
-      <wheel_separation>${wheel_base}</wheel_separation>
+      <wheel_separation>${wheel_base}</wheel_separation>     <!--see if this is track_width -->
+      <!-- <track_width>${track_width}</track_width> -->
       <wheel_radius>${wheel_radius}</wheel_radius>
       <enable_odometry>true</enable_odometry>
